File: boards/stm32-blinky/state_snapshots/pre-route/kicad/stm32-blinky.kicad_pcb (KiCad board)
At the start: 2 copper layers, 50 x 40 mm, 20 parts, among them J1 1x2 2.54mm male THT, J2 1x4 2.54mm male THT, U1 STM32F103C8T6, U2 AMS1117-3.3, Y1 8MHz 20pF

Commit message: ai-ee stm32-blinky: drc_routed pass (attempt 2, post P7->P6 relief)
Parts:
- moved C2 1.00 mm to (52.3, 42.2)
- moved C3 1.00 mm to (53.5, 33.0)
- moved R2 1.00 mm to (47.1, 31.0)
- moved U1 1.00 mm to (48.3, 37.0)
Routing:
- net +3V3: track 113.4 -> 0.00 mm
- net +5V: track 22.7 -> 0.00 mm
- net /OSC_IN: track 21.5 -> 0.00 mm
- net GND: track 20.9 -> 0.00 mm, vias 16 -> 0
- net /LED: track 19.2 -> 0.00 mm, vias 2 -> 0
- net /SWDIO: track 18.5 -> 0.00 mm
- net /OSC_OUT: track 12.0 -> 0.00 mm
- net /NRST: track 11.9 -> 0.00 mm, vias 2 -> 0
- net /LED_A: track 10.1 -> 0.00 mm
- net /SWCLK: track 6.72 -> 0.00 mm
- net /VIN: track 6.26 -> 0.00 mm
- net /BOOT0: track 1.99 -> 0.00 mm
- removed copper zone on B.Cu, net GND
