File: boards/usb-buck/state_snapshots/pre-underpass/kicad/usb-buck.kicad_pcb (KiCad board)
At the start: 4 copper layers, 50 x 40 mm, 28 parts, among them J1 USB Micro-B receptacle SMD, J2 1x4 2.54mm male THT, SW1 SMD tactile switch, U1 STM32F103C8T6, U2 AP63203QWU-7, U3 USBLC6-2SC6, Y1 8MHz 20pF

Commit message: ai-ee usb-buck: drc_routed pass (4L chain; 4 router-found defects fixed in-run)
Routing:
- net /USB_DM: track 12.4 -> 12.0 mm, vias 0 -> 2
- net VBUS: track 28.0 -> 28.1 mm, vias 2 -> 0
Changed lines of the file:
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@@
 	)
 	(segment
-		(start 23.65 32)
-		(end 27.2 28.45)
-		(width 0.3)
-		(layer "F.Cu")
-		(net "VBUS")
-	)
-	(segment
-		(start 22.6 34)
-		(end 21.7 34)
+		(start 27.2 28.45)
+		(end 22.35 33.3)
 		(width 0.3)
 		(layer "F.Cu")
@@
 	)
 	(segment
+		(start 22.35 33.3)
+		(end 22.35 33.7)
+		(width 0.3)
+		(layer "F.Cu")
+		(net "VBUS")
+	)
+	(segment
 		(start 29.1 26.55)
 		(end 29.1 28.05)
@@
 	)
 	(segment
+		(start 22.35 33.7)
+		(end 21.8 34.25)
+		(width 0.3)
+		(layer "F.Cu")
+		(net "VBUS")
+	)
+	(segment
 		(start 30.95 23.7)
 		(end 31.45 23.2)
@@
 		(width 0.3)
 		(layer "F.Cu")
-		(net "VBUS")
-	)
-	(via
-		(at 22.6 32)
-		(size 0.6)
-		(drill 0.3)
-		(layers "F.Cu" "B.Cu")
-		(net "VBUS")
-	)
-	(via
-		(at 22.6 34)
-		(size 0.6)
-		(drill 0.3)
-		(layers "F.Cu" "B.Cu")
-		(net "VBUS")
-	)
-	(segment
-		(start 22.6 32)
-		(end 22.6 34)
-		(width 0.3)
-		(layer "B.Cu")
 		(net "VBUS")
 	)
@@
 	)
 	(segment
-		(start 23.35 34.564)
-		(end 23.013 34.564)
-		(width 0.314)
-		(layer "F.Cu")
-		(net "/USB_DM")
-	)
-	(segment
-		(start 23.35 33.3)
-		(end 23.35 34.564)
-		(width 0.314)
-		(layer "F.Cu")
-		(net "/USB_DM")
-	)
-	(segment
 		(start 25.9492 34.5638)
 		(end 26.2661 34.5638)
@@
 	)
 	(segment
-		(start 21.4 33.3)
-		(end 23.35 33.3)
-		(width 0.314)
-		(layer "F.Cu")
-		(net "/USB_DM")
-	)
-	(segment
 		(start 16.33 33.31)
 		(end 17.2153 33.31)
+		(width 0.314)
+		(layer "F.Cu")
+		(net "/USB_DM")
+	)
+	(segment
+		(start 21.4 33.3)
+		(end 21.4 33.16)
 		(width 0.314)
 		(layer "F.Cu")
@@
 		(net "/USB_DM")
 	)
+	(segment
+		(start 21.4 33.16)
+		(end 21.8748 32.6852)
+		(width 0.314)
+		(layer "F.Cu")
+		(net "/USB_DM")
+	)
+	(via
+		(at 23.0128 34.5638)
+		(size 0.45)
+		(drill 0.2)
+		(layers "F.Cu" "B.Cu")
+		(net "/USB_DM")
+	)
+	(via
+		(at 21.8748 32.6852)
+		(size 0.45)
+		(drill 0.2)
+		(layers "F.Cu" "B.Cu")
+		(net "/USB_DM")
+	)
+	(segment
+		(start 21.8748 32.6852)
+		(end 21.8748 33.4258)
+		(width 0.314)
+		(layer "B.Cu")
+		(net "/USB_DM")
+	)
+	(segment
+		(start 21.8748 33.4258)
+		(end 23.0128 34.5638)
+		(width 0.314)
+		(layer "B.Cu")
+		(net "/USB_DM")
+	)
