File: boards/pd-trigger/state_snapshots/pre-stitch/kicad/pd-trigger.kicad_pcb (KiCad board)
At the start: 2 copper layers, 48 x 30 mm, 30 parts, among them J1 USB-C 16P 5A, J2 SCREW 5.08 2P, J3 HDR 1x2 AUX, Q1 BC847BS, SW1 DIP-3, U1 CH224K

Commit message: ai-ee pd-trigger: drc_routed pass (pour fan-in, 3mm trunk, netclass split)
Routing:
- net GND: track 27.2 -> 24.1 mm, vias 23 -> 15
Changed lines of the file:
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@@
-	)
-	(segment
-		(start 19.75 48.18)
-		(end 19.75 49.4)
-		(width 0.3)
-		(layer "F.Cu")
-		(net "GND")
 	)
 	(segment
@@
 	)
 	(segment
-		(start 20.4 48.18)
-		(end 20.4 48.83)
-		(width 0.3)
-		(layer "F.Cu")
-		(net "GND")
-	)
-	(segment
 		(start 27.75 54.7)
 		(end 27.75 53.8134)
@@
 	)
 	(segment
-		(start 21.05 48.18)
-		(end 21.05 49.4)
-		(width 0.3)
-		(layer "F.Cu")
-		(net "GND")
-	)
-	(segment
 		(start 42.1 29.15)
 		(end 42.1 27.9959)
@@
 	)
 	(via
-		(at 21.05 49.4)
-		(size 0.6)
-		(drill 0.3)
-		(layers "F.Cu" "B.Cu")
-		(net "GND")
-	)
-	(via
-		(at 24.24 51)
-		(size 0.6)
-		(drill 0.3)
-		(layers "F.Cu" "B.Cu")
-		(net "GND")
-	)
-	(via
 		(at 28.488 47.7365)
 		(size 0.6)
@@
 	)
 	(via
-		(at 17.281 46.259)
-		(size 0.6)
-		(drill 0.3)
-		(layers "F.Cu" "B.Cu")
-		(net "GND")
-	)
-	(via
 		(at 18.878 45.814)
 		(size 0.6)
@@
 	)
 	(via
-		(at 36.689 28.59)
-		(size 0.6)
-		(drill 0.3)
-		(layers "F.Cu" "B.Cu")
-		(net "GND")
-	)
-	(via
 		(at 22 34.8)
 		(size 0.6)
@@
 	)
 	(via
-		(at 21.05 47.2)
-		(size 0.6)
-		(drill 0.3)
-		(layers "F.Cu" "B.Cu")
-		(net "GND")
-	)
-	(via
 		(at 47.7 56.4754)
 		(size 0.6)
@@
 	)
 	(via
-		(at 20.4 48.83)
-		(size 0.6)
-		(drill 0.3)
-		(layers "F.Cu" "B.Cu")
-		(net "GND")
-	)
-	(via
-		(at 17.281 38.761)
-		(size 0.6)
-		(drill 0.3)
-		(layers "F.Cu" "B.Cu")
-		(net "GND")
-	)
-	(via
 		(at 18.878 48.5367)
 		(size 0.6)
@@
 	(via
 		(at 22 50.7462)
-		(size 0.6)
-		(drill 0.3)
-		(layers "F.Cu" "B.Cu")
-		(net "GND")
-	)
-	(via
-		(at 19.75 49.4)
 		(size 0.6)
 		(drill 0.3)
@@
 		(polygon
 			(pts
-				(xy 17.2 39.7) (xy 22.6 39.7) (xy 22.6 52) (xy 17.2 52)
+				(xy 17.2 39.7) (xy 22 39.7) (xy 22 52) (xy 17.2 52)
 			)
 		)
