File: boards/lumina-carrier/kicad/eth.kicad_sch (KiCad schematic)
At the start: 21 parts, among them U10 W5500, Y10 25MHz 18pF CL crystal

Commit message: ai-ee lumina-carrier: P4 reviewer triage - 7 fixes, BOM resync, ICD rev A6, waivers
Parts:
- added C41: 100nF 50V X7R 0603, aiee:C0603, symbol aiee:CC0603KRX7R9BB104
Connections:
- net +3V3: now also C41.1
- net GND: now also C41.2
