File: boards/lumina-carrier/kicad/mcu.kicad_sch (KiCad schematic)
At the start: 13 parts, among them J2 1x6 2.54mm header (recovery), SW1 SMD tactile switch, U30 ESP32-S3-WROOM-1-N8

Commit message: ai-ee lumina-carrier: P4 reviewer triage - 7 fixes, BOM resync, ICD rev A6, waivers
Parts:
- added D31, D32: PESD3V3L1BA 3.3V ESD clamp SOD-323, aiee:SOD-323_L1.7-W1.3-LS2.6-BI, symbol aiee:PESD3V3L1BA_C2687129
- added R103, R104, R105: 1k 1% 0603, aiee:R0603, symbol aiee:0603WAF1001T5E
- added R106: 10k 1% 0603, aiee:R0603, symbol aiee:0603WAF1002T5E
Connections:
- net ENABLE: now also R103.1; no longer U30.29 (IO36)
- net FAULT: now also R104.1; no longer U30.30 (IO37)
- net GND: now also D31.2, D32.2, R106.2
- net IMON: now also R105.1; no longer U30.12 (IO8)
- net IO3_STRAP: now reaches U30.15 (IO3)
- net IO3_STRAP: now also R106.1
- new net ENABLE_M: D31.1, R103.2, U30.29 (IO36)
- new net FAULT_M: D32.1, R104.2, U30.30 (IO37)
- new net IMON_M: R105.2, U30.12 (IO8)
- no-connect marks 5 -> 4
