File: boards/lumina-carrier/kicad/expansion.kicad_sch (KiCad schematic)
At the start: 13 parts, among them J3 DS1021-2x7SF11-B 2x7 male hea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, J4 DS1021-2x12SF11-B 2x12 male h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

Commit message: ai-ee lumina-carrier: P7 partial - planes, rule areas, MDI pairs, thermal stitching (177 unrouted)
Parts:
- H5: now left out of the parts list
Changed lines of the file:
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@@
 		(unit 1)
 		(exclude_from_sim no)
-		(in_bom yes)
+		(in_bom no)
 		(on_board yes)
 		(dnp no)
