File: boards/lumina-carrier/kicad/lumina-carrier.kicad_pcb (KiCad board)
At the start: 4 copper layers, 100 x 80 mm, 116 parts, among them J1 LPJG0926HENL PoE+ RJ45 magjack, J2 1x6 2.54mm header (recovery), J3 DS1021-2x7SF11-B 2x7 male hea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, J4 DS1021-2x12SF11-B 2x12 male h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, SW1 SMD tactile switch, U1 TPS2378DDAR, U10 W5500, U20 SCT2A25STER, U21 TPS563201DDCR, U22 TPS16630PWPR, U30 ESP32-S3-WROOM-1-N8, Y10 25MHz 18pF CL crystal

Commit message: ai-ee lumina-carrier: all four H4 actions done - LED_Y_A rerouted, 188 tracks off the fab floor, 3 new DRU rules proven live
LED_Y_A vs POE_TAP_A2: 0.2031 -> 1.1500 mm, 226 pairs under 0.635 -> 0.
Track widths: 188 @ 0.1000 mm -> 187 @ 0.110 + 1 @ 0.1071; gate dfm 193 -> 5 errors.
New rules: aiee_track_width_floor (0.1016), hv_tap_general_clearance (0.600),
hv_to_netless_conductor (0.600) - each proven live by a tightening probe.
Both clearance rules scoped per refdes/layer after all 26 initial firings were
shown to be package lead frames or inner-layer plane antipads, not defects.
drc_routed 0/0. verify 119 (was 118; +2 newly-visible oscillator return-path).

Co-Authored-By: Claude Opus 5 <noreply@anthropic.com>
Claude-Session: https://claude.ai/code/session_01D8R2zBxobH9SDJBykzWLKS
Routing:
- net /poe/LED_Y_A: track 66.9 -> 69.6 mm, vias 2 -> 4

Commit message: ai-ee lumina-carrier: P9 dfm gate PASS (5 -> 0 errors), P10 package + real API quote 62.70 USD/15pcs
Both DFM defects were generator output, invisible to DRC because .kicad_pro shipped
min_hole_to_hole 0.25 mm at severity warning against JLC's 0.5 mm - the second
sub-fab floor after min_track_width. Raised to 0.5/error; drc_routed still 0/0.
API: gerber sha256 verified, audit clean (red[] yellow[] empty), JLC read back
100.0 x 80.0 mm. qty 14 rejected (pcb_qty_error 2103) - JLC uses standard steps, so 15.
Manual assembly totalled in fab/assembly-manual-work.md: 6 THT parts, 72 joints;
the 'hand-fitted magjack' is corrected - J1 is wave-soldered.

Co-Authored-By: Claude Opus 5 <noreply@anthropic.com>
Claude-Session: https://claude.ai/code/session_01D8R2zBxobH9SDJBykzWLKS
Routing:
- net +3V3: track 62.0 -> 63.3 mm, vias 40 -> 39
Changed lines of the file:
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@@
+	)
+	(via
+		(at 44.65 96.65)
+		(size 0.6)
+		(drill 0.3)
+		(layers "F.Cu" "B.Cu")
+		(net "GND")
 	)
 	(via
@@
 	)
 	(via
-		(at 44.46 96.46)
-		(size 0.6)
-		(drill 0.3)
-		(layers "F.Cu" "B.Cu")
-		(net "GND")
-	)
-	(via
 		(at 104.95 81)
 		(size 0.6)
@@
 	(segment
 		(start 97.6312 84.8127)
+		(end 98.3 84.3)
+		(width 0.5)
+		(layer "F.Cu")
+		(net "+3V3")
+	)
+	(segment
+		(start 97.6312 84.8127)
 		(end 97.65 84.8)
 		(width 0.5)
@@
 		(end 99.675 77.675)
 		(width 0.2)
+		(layer "F.Cu")
+		(net "+3V3")
+	)
+	(segment
+		(start 98.3 84.3)
+		(end 98.65 84.1)
+		(width 0.5)
 		(layer "F.Cu")
 		(net "+3V3")
@@
 		(size 0.6)
 		(drill 0.3)
-		(layers "F.Cu" "B.Cu")
-		(net "+3V3")
-	)
-	(via
-		(at 98.091 84.353)
-		(size 0.6)
-		(drill 0.3)
