File: boards/lumina-carrier/work/p7/hvtest/lumina-carrier.kicad_pcb (KiCad board)
At the start: 4 copper layers, 100 x 80 mm, 116 parts, among them J1 LPJG0926HENL PoE+ RJ45 magjack, J2 1x6 2.54mm header (recovery), J3 DS1021-2x7SF11-B 2x7 male hea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, J4 DS1021-2x12SF11-B 2x12 male h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, SW1 SMD tactile switch, U1 TPS2378DDAR, U10 W5500, U20 SCT2A25STER, U21 TPS563201DDCR, U22 TPS16630PWPR, U30 ESP32-S3-WROOM-1-N8, Y10 25MHz 18pF CL crystal

Commit message: ai-ee lumina-carrier: P7 partial - planes, rule areas, MDI pairs, thermal stitching (177 unrouted)
Routing:
- net /ETH_RXN: track 70.4 -> 0.00 mm, vias 2 -> 0
- net /ETH_RXP: track 65.7 -> 0.00 mm, vias 2 -> 0
- net /ETH_TXP: track 63.7 -> 0.00 mm, vias 2 -> 0
- net /ETH_TXN: track 55.9 -> 0.00 mm, vias 2 -> 0
- net GND: track 9.60 -> 0.00 mm, vias 96 -> 37
- net V48_RAW: track 0.00 -> 6.28 mm
- net +3V3: track 5.20 -> 0.00 mm, vias 31 -> 3
- net +48V_SW: track 0.00 -> 3.14 mm
