File: boards/lumina-carrier/work/p7/krtf_final.kicad_pcb (KiCad board)
At the start: 4 copper layers, 100 x 80 mm, 116 parts, among them J1 LPJG0926HENL PoE+ RJ45 magjack, J2 1x6 2.54mm header (recovery), J3 DS1021-2x7SF11-B 2x7 male hea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, J4 DS1021-2x12SF11-B 2x12 male h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, SW1 SMD tactile switch, U1 TPS2378DDAR, U10 W5500, U20 SCT2A25STER, U21 TPS563201DDCR, U22 TPS16630PWPR, U30 ESP32-S3-WROOM-1-N8, Y10 25MHz 18pF CL crystal

Commit message: ai-ee lumina-carrier: P7 barrier 47->0 (1.42mm measured), unconnected 38->5, pad-shape record settled
Routing:
- net /ENABLE: track 94.6 -> 30.7 mm, vias 9 -> 5
- net /I2C_SCL: track 52.2 -> 23.0 mm, vias 9 -> 3
