File: boards/lumina-carrier/work/p7/krtf_pwr.kicad_pcb (KiCad board)
At the start: 4 copper layers, 100 x 80 mm, 116 parts, among them J1 LPJG0926HENL PoE+ RJ45 magjack, J2 1x6 2.54mm header (recovery), J3 DS1021-2x7SF11-B 2x7 male hea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, J4 DS1021-2x12SF11-B 2x12 male h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, SW1 SMD tactile switch, U1 TPS2378DDAR, U10 W5500, U20 SCT2A25STER, U21 TPS563201DDCR, U22 TPS16630PWPR, U30 ESP32-S3-WROOM-1-N8, Y10 25MHz 18pF CL crystal

Commit message: ai-ee lumina-carrier: P7 barrier 47->0 (1.42mm measured), unconnected 38->5, pad-shape record settled
Routing:
- net /ENABLE: track 94.6 -> 18.8 mm, vias 9 -> 3
- net /FAULT: track 86.3 -> 16.2 mm, vias 6 -> 4
- net /PWM0: track 62.7 -> 0.00 mm, vias 1 -> 0
- net /PWM3: track 53.0 -> 0.00 mm, vias 3 -> 0
- net /mcu/ENABLE_M: track 67.7 -> 15.7 mm, vias 3 -> 2
- net +3V3: track 62.2 -> 110.6 mm, vias 38 -> 36
- net /mcu/BOOT: track 93.6 -> 52.2 mm, vias 9 -> 4
- net /mcu/IO3_STRAP: track 39.9 -> 0.00 mm, vias 4 -> 0
- net /PWM6: track 32.6 -> 58.5 mm, vias 0 -> 1
- net /PWM2: track 63.9 -> 56.3 mm
- net /PWM4: track 55.6 -> 63.1 mm, vias 1 -> 2
- net V48_RAW: track 114.7 -> 109.7 mm
- net /mcu/RXD0: track 0.28 -> 4.83 mm, vias 0 -> 1
- net /IMON: track 55.1 -> 50.7 mm, vias 4 -> 6
- net +12V: track 111.6 -> 108.0 mm
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