File: boards/lumina-carrier/work/p7/pre_krtfinish.kicad_pcb (KiCad board)
At the start: 4 copper layers, 100 x 80 mm, 116 parts, among them J1 LPJG0926HENL PoE+ RJ45 magjack, J2 1x6 2.54mm header (recovery), J3 DS1021-2x7SF11-B 2x7 male hea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, J4 DS1021-2x12SF11-B 2x12 male h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, SW1 SMD tactile switch, U1 TPS2378DDAR, U10 W5500, U20 SCT2A25STER, U21 TPS563201DDCR, U22 TPS16630PWPR, U30 ESP32-S3-WROOM-1-N8, Y10 25MHz 18pF CL crystal

Commit message: ai-ee lumina-carrier: P7 barrier 47->0 (1.42mm measured), unconnected 38->5, pad-shape record settled
Routing:
- net /ENABLE: track 94.6 -> 18.8 mm, vias 9 -> 3
- net /ETH_LED_ACT: track 71.8 -> 0.00 mm, vias 1 -> 0
- net /FAULT: track 86.3 -> 16.2 mm, vias 6 -> 4
- net /poe/LED_Y_A: track 66.9 -> 0.00 mm, vias 2 -> 0
- net /ETH_LED_LINK: track 64.1 -> 0.00 mm, vias 2 -> 0
- net /PWM2: track 63.9 -> 0.00 mm, vias 1 -> 0
- net /PWM0: track 62.7 -> 0.00 mm, vias 1 -> 0
- net /PWM1: track 56.4 -> 0.00 mm, vias 3 -> 0
- net /PWM4: track 55.6 -> 0.00 mm, vias 1 -> 0
- net /PWM5: track 54.7 -> 0.00 mm, vias 5 -> 0
- net /mcu/TXD0: track 53.5 -> 0.00 mm, vias 1 -> 0
- net /PWM3: track 53.0 -> 0.00 mm, vias 3 -> 0
- net /mcu/ENABLE_M: track 67.7 -> 15.6 mm, vias 3 -> 2
- net /mcu/FAULT_M: track 57.2 -> 7.42 mm, vias 2 -> 0
- net /mcu/BOOT: track 93.6 -> 52.2 mm, vias 9 -> 4
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