File: boards/lumina-carrier/work/p7/krtf_r2.kicad_pcb (KiCad board)
At the start: 4 copper layers, 100 x 80 mm, 116 parts, among them J1 LPJG0926HENL PoE+ RJ45 magjack, J2 1x6 2.54mm header (recovery), J3 DS1021-2x7SF11-B 2x7 male hea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, J4 DS1021-2x12SF11-B 2x12 male h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, SW1 SMD tactile switch, U1 TPS2378DDAR, U10 W5500, U20 SCT2A25STER, U21 TPS563201DDCR, U22 TPS16630PWPR, U30 ESP32-S3-WROOM-1-N8, Y10 25MHz 18pF CL crystal

Commit message: ai-ee lumina-carrier: P7 COMPLETE - drc_routed PASS, 100% routed, 0 err 0 warn
Routing:
- net /FAULT: track 189.2 -> 83.9 mm, vias 11 -> 6
- net /ADC0: track 102.8 -> 15.8 mm, vias 10 -> 2
- net /mcu/ENABLE_M: track 66.3 -> 15.8 mm, vias 4 -> 2
- net /ETH_RSTn: track 49.3 -> 61.0 mm, vias 4 -> 6
- net /PWM3: track 53.0 -> 64.3 mm, vias 3 -> 1
- net /PWM0: track 62.7 -> 72.2 mm, vias 1 -> 5
- net /mcu/IO3_STRAP: track 40.4 -> 34.3 mm, vias 8 -> 7
- net /mcu/RXD0: track 57.9 -> 52.9 mm, vias 4 -> 2
- net /PWM1: track 56.4 -> 60.4 mm, vias 3 -> 1
- net GND: track 82.4 -> 79.2 mm, vias 104 -> 103
- net /eth/EXRES: track 15.8 -> 14.0 mm
- net /mcu/TXD0: track 52.7 -> 52.8 mm, vias 1 -> 3
