File: boards/lumina-carrier/work/p7/snap_r0_c35moved.kicad_pcb (KiCad board)
At the start: 4 copper layers, 100 x 80 mm, 116 parts, among them J1 LPJG0926HENL PoE+ RJ45 magjack, J2 1x6 2.54mm header (recovery), J3 DS1021-2x7SF11-B 2x7 male hea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, J4 DS1021-2x12SF11-B 2x12 male h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, SW1 SMD tactile switch, U1 TPS2378DDAR, U10 W5500, U20 SCT2A25STER, U21 TPS563201DDCR, U22 TPS16630PWPR, U30 ESP32-S3-WROOM-1-N8, Y10 25MHz 18pF CL crystal

Commit message: ai-ee lumina-carrier: P7 COMPLETE - drc_routed PASS, 100% routed, 0 err 0 warn
Parts:
- moved C35 0.30 mm to (97.6, 85.8)
Routing:
- net /FAULT: track 189.2 -> 86.3 mm, vias 11 -> 6
- net /ADC0: track 102.8 -> 15.8 mm, vias 10 -> 2
- net /mcu/RXD0: track 57.9 -> 0.28 mm, vias 4 -> 0
- net /mcu/STATUS: track 45.1 -> 1.47 mm, vias 4 -> 2
- net GND: track 82.4 -> 79.2 mm, vias 104 -> 103
- net /mcu/BOOT: track 91.8 -> 93.6 mm, vias 6 -> 9
- net /eth/EXRES: track 15.8 -> 14.0 mm
- net /mcu/ENABLE_M: track 66.3 -> 67.7 mm, vias 4 -> 3
- net /mcu/TXD0: track 52.7 -> 53.5 mm
- net /ETH_RSTn: track 49.3 -> 49.8 mm, vias 4 -> 6
- net /mcu/IO3_STRAP: track 40.4 -> 39.9 mm, vias 8 -> 4
