File: boards/lumina-par/state_snapshots/pre-fix-erc-a1-review/kicad/control.kicad_sch (KiCad schematic)
At the start: 39 parts, among them J4 DS1023-2*12SF11 2x12 socket, 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, U201 SN74LVC1G08DBVR single 2-inpu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, U202 SN74LVC00ADR quad 2-input NAN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, U203 M24C32-WMN6TP 32 kbit I2C EEP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, U204 SN74LVC14ADR hex Schmitt-trig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

Commit message: ai-ee lumina-par: erc pass after P4 review fixes (E-1 COFF values, E-2 NTC protection, E-3 DRV_EN pull-downs)
Parts:
- removed R218, R219, R220, R221: 10k 0603 1%, aiee:R0603, symbol aiee:0603WAF1002T5E
Other:
- note removed: "R218-R221 = 10k /DRV_ENn pull-downs, FITTED. NOT 100k: the TPS92515HV PWM pin sources 25 uA, so 100k rests at 2.5 V and latches the driver ON."
