File: boards/lumina-par/state_snapshots/p7-pre-lastmile-2/kicad/lumina-par.kicad_pcb (KiCad board)
At the start: 4 copper layers, 100 x 80 mm, 159 parts, among them J3 DS1023-2*7SF11 2x7 socket 2.5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, J4 DS1023-2*12SF11 2x12 socket, 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, J5 S10B-PH-SM4-TB JST PH 10-way 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, Q101 NCE01P13K -100V P-MOSFET TO-2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, Q102 BSS123 100V N-MOSFET SOT-23, Q301 SSM3K2615R 60V 2A N-FET, Q321 SSM3K2615R 60V 2A N-FET, Q341 SSM3K2615R 60V 2A N-FET, Q361 SSM3K2615R 60V 2A N-FET, U201 SN74LVC1G08DBVR single 2-inpu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, U202 SN74LVC00ADR quad 2-input NAN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, U203 M24C32-WMN6TP 32 kbit I2C EEP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, U204 SN74LVC14ADR hex Schmitt-trig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, U301 TPS92515HVDGQR, U321 TPS92515HVDGQR, U341 TPS92515HVDGQR, U361 TPS92515HVDGQR, U401 LM339LVPWR quad open-drain co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

Commit message: ai-ee lumina-par: drc_routed pass - 100% routed, 0 violations
Routing:
- net /EN_OK: track 116.6 -> 78.5 mm, vias 7 -> 4
- net /ADC0: track 60.4 -> 43.7 mm, vias 5 -> 4
- net /NTC_LED: track 114.9 -> 102.7 mm, vias 6 -> 5
- net GND: track 64.8 -> 58.2 mm, vias 119 -> 118
- net +3V3: track 270.9 -> 267.6 mm, vias 14 -> 13
Changed lines of the file:
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@@
 	)
 	(segment
-		(start 146.65 124.3)
-		(end 146.65 123.15)
-		(width 0.2)
-		(layer "F.Cu")
-		(net "GND")
-	)
-	(segment
 		(start 146.7 115.5)
 		(end 146.75 115.45)
@@
 	)
 	(via
-		(at 146.65 123.15)
-		(size 0.45)
-		(drill 0.2)
-		(layers "F.Cu" "B.Cu")
-		(net "GND")
-	)
-	(via
 		(at 135.6 114.95)
 		(size 0.6)
@@
 	)
 	(segment
-		(start 146.65 123.15)
-		(end 143.5 118.7)
-		(width 0.2)
-		(layer "In2.Cu")
-		(net "GND")
-	)
-	(segment
 		(start 138.5 123.7)
 		(end 146.7 115.5)
@@
 	)
 	(segment
-		(start 133 106.21)
-		(end 133 110)
-		(width 0.2)
-		(layer "F.Cu")
-		(net "/EN_OK")
-	)
-	(segment
 		(start 103.65 85.2)
 		(end 103.6 85.25)
@@
 	)
 	(segment
-		(start 130.38 106.21)
-		(end 135.62 106.21)
-		(width 0.2)
-		(layer "F.Cu")
-		(net "/EN_OK")
-	)
-	(segment
 		(start 82.2 99.75)
 		(end 78.75 99.75)
@@
 	)
 	(segment
-		(start 111.75 85.75)
-		(end 111.75 87.5)
-		(width 0.2)
-		(layer "F.Cu")
-		(net "/EN_OK")
-	)
-	(segment
 		(start 89.35 90.9)
 		(end 86.75 93.5)
@@
 	)
 	(segment
-		(start 134.7 124)
-		(end 134.7 125.2)
-		(width 0.2)
-		(layer "F.Cu")
-		(net "/EN_OK")
-	)
-	(segment
 		(start 130.4 110)
 		(end 135.6 110)
@@
 	)
 	(via
-		(at 111.75 87.5)
-		(size 0.45)
-		(drill 0.2)
-		(layers "F.Cu" "B.Cu")
-		(net "/EN_OK")
-	)
-	(via
-		(at 135 117.1)
-		(size 0.45)
-		(drill 0.2)
-		(layers "F.Cu" "B.Cu")
-		(net "/EN_OK")
-	)
-	(via
 		(at 101.2 87.75)
 		(size 0.45)
@@
 		(net "/EN_OK")
 	)
-	(via
-		(at 134.7 124)
-		(size 0.45)
-		(drill 0.2)
-		(layers "F.Cu" "B.Cu")
-		(net "/EN_OK")
-	)
-	(segment
-		(start 135 117.1)
-		(end 134.7 124)
-		(width 0.2)
-		(layer "B.Cu")
-		(net "/EN_OK")
-	)
 	(segment
 		(start 99.65 89.8)
@@
 	)
 	(segment
-		(start 135 110.5)
-		(end 135 117.1)
-		(width 0.2)
-		(layer "In2.Cu")
-		(net "/EN_OK")
-	)
-	(segment
 		(start 122.85 102.45)
 		(end 123.95 103.55)
@@
 	)
 	(segment
-		(start 111.75 87.5)
-		(end 106.1 93.15)
-		(width 0.2)
-		(layer "In2.Cu")
-		(net "/EN_OK")
-	)
-	(segment
 		(start 125.6 106.2)
 		(end 125.6 106.5)
@@
 	)
 	(segment
-		(start 130.4 109.9)
-		(end 135 110.5)
-		(width 0.2)
-		(layer "In2.Cu")
-		(net "/EN_OK")
-	)
-	(segment
 		(start 104.5 91.5)
 		(end 104.55 91.55)
@@
 	)
 	(segment
-		(start 145.2753 113.1365)
-		(end 146.15 113.05)
-		(width 0.2)
-		(layer "F.Cu")
-		(net "+3V3")
-	)
-	(segment
 		(start 132.7 125.3)
 		(end 131.8 124.4)
@@
 	)
 	(via
-		(at 146.15 113.05)
-		(size 0.45)
-		(drill 0.2)
-		(layers "F.Cu" "B.Cu")
-		(net "+3V3")
-	)
-	(via
 		(at 144.9 115.2)
 		(size 0.45)
@@
 	)
 	(segment
-		(start 146.15 113.05)
-		(end 144.45 114.75)
-		(width 0.2)
-		(layer "In1.Cu")
-		(net "+3V3")
-	)
-	(segment
 		(start 134.55 122.85)
 		(end 134.45 122.85)
@@
 	)
 	(segment
-		(start 143.7753 113.1365)
-		(end 142.4 113.6)
-		(width 0.2)
-		(layer "F.Cu")
-		(net "/NTC_LED")
-	)
-	(segment
 		(start 111.5 111.55)
 		(end 111.75 111.55)
@@
 	)
 	(via
-		(at 142.4 113.6)
-		(size 0.45)
-		(drill 0.2)
-		(layers "F.Cu" "B.Cu")
-		(net "/NTC_LED")
-	)
-	(via
 		(at 103.3 99)
 		(size 0.45)
@@
 	)
 	(segment
-		(start 140 115.2)
-		(end 139.8 118)
-		(width 0.2)
-		(layer "In1.Cu")
-		(net "/NTC_LED")
-	)
-	(segment
 		(start 101.6 71)
 		(end 101.65 71.05)
@@
 	)
 	(segment
-		(start 139.8 118)
-		(end 138.6 122.6)
-		(width 0.2)
-		(layer "In1.Cu")
-		(net "/NTC_LED")
-	)
-	(segment
 		(start 137.95 122.75)
 		(end 138.1 122.6)
@@
 	)
 	(segment
-		(start 141.5 113.5)
-		(end 140 115.2)
-		(width 0.2)
-		(layer "In1.Cu")
-		(net "/NTC_LED")
-	)
-	(segment
-		(start 142.4 113.6)
-		(end 141.5 113.5)
-		(width 0.2)
-		(layer "In1.Cu")
-		(net "/NTC_LED")
-	)
-	(segment
 		(start 133.55 121.75)
 		(end 133.7 121.9)
@@
 	)
 	(segment
-		(start 139.9 118)
-		(end 137.3 118)
-		(width 0.2)
-		(layer "F.Cu")
-		(net "/ADC0")
-	)
-	(segment
 		(start 115.525 121.85)
 		(end 115.475 121.8)
@@
 	)
 	(segment
-		(start 140.3326 119.0733)
-		(end 139.9 118)
-		(width 0.2)
-		(layer "F.Cu")
-		(net "/ADC0")
-	)
-	(segment
 		(start 117.225 122)
 		(end 115.95 122)
@@
 		(net "/ADC0")
 	)
-	(via
-		(at 137.3 118)
-		(size 0.45)
-		(drill 0.2)
-		(layers "F.Cu" "B.Cu")
-		(net "/ADC0")
-	)
 	(segment
 		(start 112.75 117.7)
@@
 	)
 	(segment
-		(start 133.1 123.2)
-		(end 132.1 124.9)
-		(width 0.2)
-		(layer "In2.Cu")
-		(net "/ADC0")
-	)
-	(segment
 		(start 104.5 110.275)
 		(end 104.5 106.775)
@@
 		(width 0.2)
 		(layer "In2.Cu")
-		(net "/ADC0")
-	)
-	(segment
-		(start 132.1 124.9)
-		(end 132.025 129.125)
-		(width 0.2)
-		(layer "In2.Cu")
-		(net "/ADC0")
-	)
-	(segment
-		(start 137.3 118)
-		(end 133.1 123.2)
-		(width 0.2)
-		(layer "In2.Cu")
