File: boards/lumina-par/state_snapshots/pre-review-fix/kicad/lumina-par.kicad_pcb (KiCad board)
At the start: 4 copper layers, 100 x 80 mm, 158 parts, among them J3 DS1023-2*7SF11 2x7 socket 2.5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, J4 DS1023-2*12SF11 2x12 socket, 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, J5 S10B-PH-SM4-TB JST PH 10-way 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, Q101 NCE01P13K -100V P-MOSFET TO-2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, Q102 BSS123 100V N-MOSFET SOT-23, Q301 SSM3K2615R 60V 2A N-FET, Q321 SSM3K2615R 60V 2A N-FET, Q341 SSM3K2615R 60V 2A N-FET, Q361 SSM3K2615R 60V 2A N-FET, U201 SN74LVC1G08DBVR single 2-inpu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, U202 SN74LVC00ADR quad 2-input NAN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, U203 M24C32-WMN6TP 32 kbit I2C EEP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, U204 SN74LVC14ADR hex Schmitt-trig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, U301 TPS92515HVDGQR, U321 TPS92515HVDGQR, U341 TPS92515HVDGQR, U361 TPS92515HVDGQR, U401 LM339LVPWR quad open-drain co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

Commit message: ai-ee lumina-par: P8 review fixes - hazard silk, mated-view pin-1 triangles, thermal vias, H1 deleted (ICD rev A8)
Routing:
- net GND: vias 131 -> 119
Other:
- board text removed: "BREAKS PD DETECTION. USE AN"
- board text removed: "ISOLATED PROBE ON EVERY TEST POINT"
- board text removed: "NO EARTH GND. AN EARTHED PROBE"
- board text removed: "PoE HAZARD"
- board text removed: "PoE HV"
- board text removed: "WARNING - FLOATS AT PoE POTENTIAL"
- board text removed: "▲"
Changed lines of the file:
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@@
 		(layer "Edge.Cuts")
-	)
-	(gr_text "PoE HV"
-		(at 57.7495 71.9995 0)
-		(layer "F.SilkS")
-		(effects
-			(font
-				(size 1 1)
-				(thickness 0.16)
-			)
-		)
-	)
-	(gr_text "WARNING - FLOATS AT PoE POTENTIAL"
-		(at 72.9375 120.2925 0)
-		(layer "F.SilkS")
-		(effects
-			(font
-				(size 1 1)
-				(thickness 0.16)
-			)
-		)
-	)
-	(gr_text "NO EARTH GND. AN EARTHED PROBE"
-		(at 72.9375 121.8925 0)
-		(layer "F.SilkS")
-		(effects
-			(font
-				(size 1 1)
-				(thickness 0.16)
-			)
-		)
-	)
-	(gr_text "BREAKS PD DETECTION. USE AN"
-		(at 72.9375 123.4925 0)
-		(layer "F.SilkS")
-		(effects
-			(font
-				(size 1 1)
-				(thickness 0.16)
-			)
-		)
-	)
-	(gr_text "ISOLATED PROBE ON EVERY TEST POINT"
-		(at 72.9375 125.0925 0)
-		(layer "F.SilkS")
-		(effects
-			(font
-				(size 1 1)
-				(thickness 0.16)
-			)
-		)
-	)
-	(gr_text "PoE HV"
-		(at 93.7495 71.9995 0)
-		(layer "F.SilkS")
-		(effects
-			(font
-				(size 1 1)
-				(thickness 0.16)
-			)
-		)
-	)
-	(gr_text "PoE HV"
-		(at 103.7495 99.2495 0)
-		(layer "F.SilkS")
-		(effects
-			(font
-				(size 1 1)
-				(thickness 0.16)
-			)
-		)
-	)
-	(gr_text "PoE HAZARD"
-		(at 150.2495 76.4425 0)
-		(layer "F.SilkS")
-		(effects
-			(font
-				(size 1 1)
-				(thickness 0.16)
-			)
-		)
-	)
-	(gr_text "▲"
-		(at 70.3165 136.5425 0)
-		(layer "B.SilkS")
-		(effects
-			(font
-				(size 0.8 0.8)
-				(thickness 0.16)
-			)
-			(justify mirror)
-		)
-	)
-	(gr_text "▲"
-		(at 111.9665 136.5425 0)
-		(layer "B.SilkS")
-		(effects
-			(font
-				(size 0.8 0.8)
-				(thickness 0.16)
-			)
-			(justify mirror)
-		)
 	)
 	(segment
@@
 	)
 	(via
-		(at 121.2805 109.8645)
-		(size 0.45)
-		(drill 0.2)
-		(layers "F.Cu" "B.Cu")
-		(net "GND")
-	)
-	(via
-		(at 128.3395 115.4505)
-		(size 0.45)
-		(drill 0.2)
-		(layers "F.Cu" "B.Cu")
-		(net "GND")
-	)
-	(via
 		(at 138.499 123.721)
 		(size 0.6)
@@
 	)
 	(via
-		(at 104.9395 114.3505)
-		(size 0.45)
-		(drill 0.2)
-		(layers "F.Cu" "B.Cu")
-		(net "GND")
-	)
-	(via
 		(at 118.7 84.85)
 		(size 0.6)
@@
 	)
 	(via
-		(at 127.9395 90.8505)
-		(size 0.45)
-		(drill 0.2)
-		(layers "F.Cu" "B.Cu")
-		(net "GND")
-	)
-	(via
 		(at 122.36 86.5)
 		(size 0.45)
@@
 		(size 0.6)
 		(drill 0.3)
-		(layers "F.Cu" "B.Cu")
-		(net "GND")
-	)
-	(via
-		(at 128.3395 91.4505)
-		(size 0.45)
-		(drill 0.2)
 		(layers "F.Cu" "B.Cu")
 		(net "GND")
@@
 	)
 	(via
-		(at 128.4395 114.3505)
-		(size 0.45)
-		(drill 0.2)
-		(layers "F.Cu" "B.Cu")
-		(net "GND")
-	)
-	(via
 		(at 99.22 111.135)
 		(size 0.45)
@@
 	)
 	(via
-		(at 104.4395 114.8505)
-		(size 0.45)
-		(drill 0.2)
-		(layers "F.Cu" "B.Cu")
-		(net "GND")
-	)
-	(via
 		(at 96.6 78.15)
 		(size 0.6)
@@
 	)
 	(via
-		(at 105.1395 90.2505)
-		(size 0.45)
-		(drill 0.2)
-		(layers "F.Cu" "B.Cu")
-		(net "GND")
-	)
-	(via
 		(at 116.998 65.015)
 		(size 0.6)
@@
 	)
 	(via
-		(at 127.9395 114.8505)
-		(size 0.45)
-		(drill 0.2)
-		(layers "F.Cu" "B.Cu")
-		(net "GND")
-	)
-	(via
 		(at 56.85 98.25)
 		(size 0.6)
@@
 	)
 	(via
-		(at 104.8395 115.4505)
-		(size 0.45)
-		(drill 0.2)
-		(layers "F.Cu" "B.Cu")
-		(net "GND")
-	)
-	(via
 		(at 122 85.865)
 		(size 0.45)
@@
 	)
 	(via
-		(at 128.4395 90.3505)
-		(size 0.45)
-		(drill 0.2)
-		(layers "F.Cu" "B.Cu")
-		(net "GND")
-	)
-	(via
 		(at 122 89.51)
 		(size 0.6)
@@
 		(layers "F.Cu" "B.Cu")
 		(net "GND")
-	)
-	(via
-		(at 104.4395 90.3505)
-		(size 0.45)
-		(drill 0.2)
-		(layers "F.Cu" "B.Cu")
-		(net "GND")
