File: boards/rf-term-150w/state_snapshots/pre-fix-parity/kicad/rf-term-150w.kicad_sch (KiCad schematic)
At the start: 6 parts, among them J1 SMA

Commit message: ai-ee rf-term-150w: P5 board setup - 26x20 2L, parity 0, 10 rules
Co-Authored-By: Claude Opus 5 (1M context) <noreply@anthropic.com>
Claude-Session: https://claude.ai/code/session_01XcrCcgsAPUYzrFgzP9SkX5
Parts:
- J1: footprint aiee:SMA_BAT_Wireless_BWSMA-KWE-Z001 -> Connector_Coaxial:SMA_BAT_Wireless_BWSMA-KWE-Z001
Changed lines of the file:
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@@
 			)
 		)
-		(property "Footprint" "aiee:SMA_BAT_Wireless_BWSMA-KWE-Z001"
+		(property "Footprint" "Connector_Coaxial:SMA_BAT_Wireless_BWSMA-KWE-Z001"
 			(at 63.5 76.2 0.0000)
 			(effects
@@
 		(instances
 			(project "rf-term-150w"
-				(path "/a9517388-6a30-4643-8ce1-903b1639c51c"
+				(path "/6c097ad7-27fb-47cd-952a-76b2dd19244a"
 					(reference "J1")
 					(unit 1)
@@
 		(instances
 			(project "rf-term-150w"
-				(path "/a9517388-6a30-4643-8ce1-903b1639c51c"
+				(path "/6c097ad7-27fb-47cd-952a-76b2dd19244a"
 					(reference "#PWR01")
 					(unit 1)
@@
 			)
 		)
-		(property "Description" "Johanson 5602 air trimmer, 1-30pF 250VDC -65/+125C, top-adjust panel-mount. Pad 1=CASE/THREAD -> GND, Pad 2=LEAD -> RF (physical assignment, state.json P3 decision 2026-08-09)."
-			(at 101.6 76.2 0)
-			(effects
-				(font
-					(size 1.27 1.27)
-				)
-				(hide yes)
-			)
-		)
 		(pin "2"
 		)
@@
 		(instances
 			(project "rf-term-150w"
-				(path "/a9517388-6a30-4643-8ce1-903b1639c51c"
+				(path "/6c097ad7-27fb-47cd-952a-76b2dd19244a"
 					(reference "C1")
 					(unit 1)
@@
 		(instances
 			(project "rf-term-150w"
-				(path "/a9517388-6a30-4643-8ce1-903b1639c51c"
+				(path "/6c097ad7-27fb-47cd-952a-76b2dd19244a"
 					(reference "#PWR02")
 					(unit 1)
@@
 		(instances
 			(project "rf-term-150w"
-				(path "/a9517388-6a30-4643-8ce1-903b1639c51c"
+				(path "/6c097ad7-27fb-47cd-952a-76b2dd19244a"
 					(reference "R1")
 					(unit 1)
@@
 		(instances
 			(project "rf-term-150w"
-				(path "/a9517388-6a30-4643-8ce1-903b1639c51c"
+				(path "/6c097ad7-27fb-47cd-952a-76b2dd19244a"
 					(reference "#PWR03")
 					(unit 1)
@@
 		(instances
 			(project "rf-term-150w"
-				(path "/a9517388-6a30-4643-8ce1-903b1639c51c"
+				(path "/6c097ad7-27fb-47cd-952a-76b2dd19244a"
 					(reference "H1")
 					(unit 1)
@@
 		(instances
 			(project "rf-term-150w"
-				(path "/a9517388-6a30-4643-8ce1-903b1639c51c"
+				(path "/6c097ad7-27fb-47cd-952a-76b2dd19244a"
 					(reference "#PWR04")
 					(unit 1)
@@
 		(instances
 			(project "rf-term-150w"
-				(path "/a9517388-6a30-4643-8ce1-903b1639c51c"
+				(path "/6c097ad7-27fb-47cd-952a-76b2dd19244a"
 					(reference "H2")
 					(unit 1)
@@
 		(instances
 			(project "rf-term-150w"
-				(path "/a9517388-6a30-4643-8ce1-903b1639c51c"
+				(path "/6c097ad7-27fb-47cd-952a-76b2dd19244a"
 					(reference "#PWR05")
 					(unit 1)
@@
 		(instances
 			(project "rf-term-150w"
-				(path "/a9517388-6a30-4643-8ce1-903b1639c51c"
+				(path "/6c097ad7-27fb-47cd-952a-76b2dd19244a"
 					(reference "H3")
 					(unit 1)
@@
 		(instances
 			(project "rf-term-150w"
-				(path "/a9517388-6a30-4643-8ce1-903b1639c51c"
+				(path "/6c097ad7-27fb-47cd-952a-76b2dd19244a"
 					(reference "#PWR06")
 					(unit 1)
@@
 		(instances
 			(project "rf-term-150w"
-				(path "/a9517388-6a30-4643-8ce1-903b1639c51c"
+				(path "/6c097ad7-27fb-47cd-952a-76b2dd19244a"
 					(reference "#PWR07")
 					(unit 1)
@@
 		(instances
 			(project "rf-term-150w"
-				(path "/a9517388-6a30-4643-8ce1-903b1639c51c"
+				(path "/6c097ad7-27fb-47cd-952a-76b2dd19244a"
 					(reference "#FLG01")
 					(unit 1)
