File: boards/bb-mcu/kicad/bb-mcu.kicad_sch (KiCad schematic)
At the start: 9 parts, among them J1 2P 5.08mm screw terminal THT, J2 1x5 2.54mm male THT, J3 1x5 2.54mm male THT, U1 STM32F030F4P6TR

Commit message: ai-ee bb-mcu: erc pass (P4 review amendments - C5 NRST cap, J3 reorder)
Parts:
- added C5: 100nF 50V X7R, aiee:C0603, symbol aiee:CC0603KRX7R9BB104
Connections:
- net GND: now also J3.5, C5.2; no longer J3.3
- net IO3: now also J3.3; no longer J3.4
- net IO4: now also J3.4; no longer J3.5
- net NRST: now also C5.1
Changed lines of the file:
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@@
 		(instances
 			(project "bb-mcu"
-				(path "/967b028f-9fd4-4020-a264-bd5b379ed5ba"
+				(path "/730838dd-2da2-4635-a5fe-1720a2eeb369"
 					(reference "U1")
 					(unit 1)
@@
 		(instances
 			(project "bb-mcu"
-				(path "/967b028f-9fd4-4020-a264-bd5b379ed5ba"
+				(path "/730838dd-2da2-4635-a5fe-1720a2eeb369"
 					(reference "C1")
 					(unit 1)
@@
 		(instances
 			(project "bb-mcu"
-				(path "/967b028f-9fd4-4020-a264-bd5b379ed5ba"
+				(path "/730838dd-2da2-4635-a5fe-1720a2eeb369"
 					(reference "C2")
 					(unit 1)
@@
 		(instances
 			(project "bb-mcu"
-				(path "/967b028f-9fd4-4020-a264-bd5b379ed5ba"
+				(path "/730838dd-2da2-4635-a5fe-1720a2eeb369"
 					(reference "C3")
 					(unit 1)
@@
 		(instances
 			(project "bb-mcu"
-				(path "/967b028f-9fd4-4020-a264-bd5b379ed5ba"
+				(path "/730838dd-2da2-4635-a5fe-1720a2eeb369"
 					(reference "C4")
 					(unit 1)
@@
 		(instances
 			(project "bb-mcu"
-				(path "/967b028f-9fd4-4020-a264-bd5b379ed5ba"
+				(path "/730838dd-2da2-4635-a5fe-1720a2eeb369"
 					(reference "R1")
+					(unit 1)
+				)
+			)
+		)
+	)
+	(symbol
+		(lib_id "aiee:CC0603KRX7R9BB104")
+		(at 190.5 190.5 0)
+		(unit 1)
+		(exclude_from_sim no)
+		(in_bom yes)
+		(on_board yes)
+		(dnp no)
+		(fields_autoplaced no)
+		(property "Reference" "C5"
+			(at 189.5106 187.2 0.0000)
+			(effects
+				(font
+					(size 1.27 1.27)
+				)
+				(justify left)
+			)
+		)
+		(property "Value" "100nF 50V X7R"
+			(at 184.4814 193.8 0.0000)
+			(effects
+				(font
+					(size 1.27 1.27)
+				)
+				(justify left)
+			)
+		)
+		(property "Footprint" "aiee:C0603"
+			(at 190.5 182.88 0.0000)
+			(effects
+				(font
+					(size 1.27 1.27)
+				)
+				(hide yes)
+			)
+		)
+		(property "LCSC" "C14663"
+			(at 193.04 195.5799 0)
+			(effects
+				(font
+					(size 1.27 1.27)
+				)
+				(justify left)
+			)
+		)
+		(pin "1"
+		)
+		(pin "2"
+		)
+		(instances
+			(project "bb-mcu"
+				(path "/730838dd-2da2-4635-a5fe-1720a2eeb369"
+					(reference "C5")
 					(unit 1)
 				)
@@
 		(instances
 			(project "bb-mcu"
-				(path "/967b028f-9fd4-4020-a264-bd5b379ed5ba"
+				(path "/730838dd-2da2-4635-a5fe-1720a2eeb369"
 					(reference "J1")
 					(unit 1)
@@
 		(instances
 			(project "bb-mcu"
-				(path "/967b028f-9fd4-4020-a264-bd5b379ed5ba"
+				(path "/730838dd-2da2-4635-a5fe-1720a2eeb369"
 					(reference "J2")
 					(unit 1)
@@
 		(instances
 			(project "bb-mcu"
-				(path "/967b028f-9fd4-4020-a264-bd5b379ed5ba"
+				(path "/730838dd-2da2-4635-a5fe-1720a2eeb369"
 					(reference "J3")
 					(unit 1)
@@
 		(instances
 			(project "bb-mcu"
-				(path "/967b028f-9fd4-4020-a264-bd5b379ed5ba"
+				(path "/730838dd-2da2-4635-a5fe-1720a2eeb369"
 					(reference "#PWR01")
 					(unit 1)
@@
 		(instances
 			(project "bb-mcu"
-				(path "/967b028f-9fd4-4020-a264-bd5b379ed5ba"
+				(path "/730838dd-2da2-4635-a5fe-1720a2eeb369"
 					(reference "#FLG01")
 					(unit 1)
@@
 		(instances
 			(project "bb-mcu"
-				(path "/967b028f-9fd4-4020-a264-bd5b379ed5ba"
+				(path "/730838dd-2da2-4635-a5fe-1720a2eeb369"
 					(reference "#PWR02")
 					(unit 1)
@@
 		(instances
 			(project "bb-mcu"
-				(path "/967b028f-9fd4-4020-a264-bd5b379ed5ba"
+				(path "/730838dd-2da2-4635-a5fe-1720a2eeb369"
 					(reference "#FLG02")
 					(unit 1)
@@
 	(wire
 		(pts
+			(xy 185.42 190.5) (xy 182.88 190.5)
+		)
+		(stroke
+			(width 0)
+			(type default)
+		)
+	)
+	(wire
+		(pts
+			(xy 195.58 190.5) (xy 198.12 190.5)
+		)
+		(stroke
+			(width 0)
+			(type default)
+		)
+	)
+	(wire
+		(pts
 			(xy 74.93 106.68) (xy 74.93 109.22)
 		)
@@
 		)
 	)
+	(label "NRST"
+		(at 182.88 190.5 0.0000)
+		(effects
+			(font
+				(size 1.27 1.27)
+			)
+			(justify left bottom)
+		)
+	)
+	(label "GND"
+		(at 198.12 190.5 0.0000)
+		(effects
+			(font
+				(size 1.27 1.27)
+			)
+			(justify left bottom)
+		)
+	)
 	(label "+3V3"
 		(at 74.93 109.22 0.0000)
@@
 		)
 	)
+	(label "IO3"
+		(at 293.37 190.5 0.0000)
+		(effects
+			(font
+				(size 1.27 1.27)
+			)
+			(justify left bottom)
+		)
+	)
+	(label "IO4"
+		(at 293.37 193.04 0.0000)
+		(effects
+			(font
+				(size 1.27 1.27)
+			)
+			(justify left bottom)
+		)
+	)
 	(label "GND"
-		(at 293.37 190.5 0.0000)
-		(effects
-			(font
-				(size 1.27 1.27)
-			)
-			(justify left bottom)
-		)
-	)
-	(label "IO3"
-		(at 293.37 193.04 0.0000)
-		(effects
-			(font
-				(size 1.27 1.27)
-			)
-			(justify left bottom)
-		)
-	)
-	(label "IO4"
 		(at 293.37 195.58 0.0000)
 		(effects
