File: boards/bb-mcu/kicad/route/prefinish_bb-mcu.kicad_pcb (KiCad board)
At the start: 2 copper layers, 34.8 x 22.3 mm, 14 parts, among them J1 2P 5.08mm screw terminal THT, J2 1x5 2.54mm male THT, J3 1x5 2.54mm male THT, U1 STM32F030F4P6TR

Commit message: ai-ee bb-mcu: drc_routed pass (completion 1.0, pour unbroken)
Routing:
- net GND: track 28.8 -> 1.19 mm, vias 8 -> 1
- net /SWDIO: track 11.4 -> 0.00 mm
- net /NRST: track 9.74 -> 0.00 mm
- net /SWCLK: track 4.65 -> 0.00 mm
