File: boards/bb-ldo/state_snapshots/pre-fix-3items/kicad/bb-ldo.kicad_pcb (KiCad board)
At the start: 2 copper layers, 50 x 26.4 mm, 5 parts, among them J1 2P 5.08mm THT screw terminal, J2 2P 5.08mm THT screw terminal, U1 AMS1117-3.3

Commit message: ai-ee bb-ldo: verify pass (P8 fixes: vias out of pads, redundant GND barrels, HOT SURFACE legend)
Routing:
- net GND: track 7.60 -> 5.16 mm, vias 5 -> 4
Other:
- board text removed: "HOT SURFACE"
Changed lines of the file:
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@@
-		)
-	)
-	(gr_text "HOT SURFACE"
-		(at 36.5 42.2 0)
-		(layer "F.SilkS")
-		(effects
-			(font
-				(size 1.6 1.6)
-				(thickness 0.25)
-			)
 		)
 	)
@@
 		(net "GND")
 	)
-	(segment
-		(start 17.968 32.91)
-		(end 17.968 30.47)
-		(width 0.6)
-		(layer "F.Cu")
-		(net "GND")
-	)
 	(via
 		(at 16.325 32.91)
@@
 		(size 0.6)
 		(drill 0.3)
-		(layers "F.Cu" "B.Cu")
-		(net "GND")
-	)
-	(via
-		(at 17.968 30.47)
-		(size 0.6)
-		(drill 0.3)
