File: boards/g0-sense/state_snapshots/pre-p7-route/kicad/g0-sense.kicad_pcb (KiCad board)
At the start: 2 copper layers, 35.8 x 28.3 mm, 30 parts, among them J1 TYPE-C-31-M-12, J2 Qwiic JST SH 4P, J3 1x4 2.54mm THT (DNP), J4 1x4 2.54mm THT (DNP), SW1 Tactile button, U1 AMS1117-3.3, U2 STM32G030F6P6, U3 SHT40-AD1B-R2

Commit message: ai-ee g0-sense: run iteration 1 checkpoint
Routing:
- net /main/SCL: track 15.3 -> 0.00 mm
- net /main/SDA: track 15.2 -> 0.00 mm
- net +3V3: track 11.6 -> 0.00 mm
- net GND: track 5.22 -> 0.00 mm, vias 1 -> 0
- removed copper zone on F.Cu, net +3V3
- removed copper zone on B.Cu, net GND
- removed copper zone on F.Cu, net VBUS
