File: boards/g0-sense/state_snapshots/p7-pre-critical/kicad/g0-sense.kicad_pcb (KiCad board)
At the start: 2 copper layers, 35.8 x 28.3 mm, 30 parts, among them J1 TYPE-C-31-M-12, J2 Qwiic JST SH 4P, J3 1x4 2.54mm THT (DNP), J4 1x4 2.54mm THT (DNP), SW1 Tactile button, U1 AMS1117-3.3, U2 STM32G030F6P6, U3 SHT40-AD1B-R2

Commit message: ai-ee g0-sense: run iteration 2 checkpoint
Routing:
- net GND: track 32.3 -> 5.22 mm, vias 17 -> 1
- net /main/NRST: track 19.3 -> 0.00 mm
- net /main/UART_RX: track 18.5 -> 0.00 mm
- net /main/SCL: track 32.8 -> 15.3 mm
- net /main/SWCLK: track 12.5 -> 0.00 mm
- net /main/UART_TX: track 11.3 -> 0.00 mm
- net /main/SWDIO: track 8.82 -> 0.00 mm
- net +3V3: track 18.6 -> 11.6 mm, vias 1 -> 0
- net +5V: track 5.16 -> 0.00 mm
- net /main/SDA: track 18.1 -> 15.2 mm
- net /power/CC1: track 2.79 -> 0.00 mm
- net /power/CC2: track 2.67 -> 0.00 mm
- net /main/LED_USER: track 2.07 -> 0.00 mm
- net /main/LED_A: track 2.00 -> 0.00 mm
- net /power/PWR_LED_K: track 1.95 -> 0.00 mm
