File: boards/g0-sense/state_snapshots/pre-plane-repair/kicad/g0-sense.kicad_pcb (KiCad board)
At the start: 2 copper layers, 35.8 x 28.3 mm, 30 parts, among them J1 TYPE-C-31-M-12, J2 Qwiic JST SH 4P, J3 1x4 2.54mm THT (DNP), J4 1x4 2.54mm THT (DNP), SW1 Tactile button, U1 AMS1117-3.3, U2 STM32G030F6P6, U3 SHT40-AD1B-R2

Commit message: ai-ee g0-sense: P7 routing complete - drc_routed PASS 0/0, completion 1.0
2-layer chain: planes_gen -> route_critical -> route_auto (FR 3 rungs, best
rung 1) -> stitch_vias (13) -> plane_repair -> gate; route_cleanup skipped
per the S14 2L-pour rule.

- J1 VBUS escape resolved pour-carried (--pad-window measured the escape
  window at 1.315 mm vs the 0.8 mm rule), retiring the P6 premise that it
  was impossible: no neck, no rule exception, no via-in-pad, no JLC wicking
  remark. Two F.Cu VBUS pours joined by a 0.8 mm B.Cu bridge on 2+2 vias.
- U3 island contract met: exactly 4 necked crossings (0.127/0.127/0.127/
  0.150), zero copper and zero fill in the tongue on both layers; FR's
  fifth crossing (SCL through the island) removed, I2C trunk rebuilt on B.Cu.
  The P6 outline already carries the U-slot, so Edge.Cuts is unchanged.
- U1 tab pour 113.2 mm2 contiguous (the router's 158 mm2 is the electrical
  figure; 0.25/0.5 mm bridge tracks carry current, not heat). Accepted:
  80 C/W per AMS p5 Table 1 gives a 40.8 K rise vs the declared dt_c 45.
- Orchestrator-verified rather than taken on the agent's word: kicad-cli DRC
  0 violations / 0 unconnected / 0 parity, and plane_repair --flag-only on
  the final board shows GND B.Cu unsplit (1 group, 813.2 mm2, 27 anchors) -
  the B.Cu VBUS bridge does not sever the ground return.

Gates: erc, place, drc_routed all PASS and fresh at board hash 0b12cafc.

Co-Authored-By: Claude Opus 5 <noreply@anthropic.com>
Routing:
- net +3V3: track 89.2 -> 18.6 mm
- net VBUS: track 7.10 -> 0.00 mm, vias 4 -> 0
Changed lines of the file:
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@@
-	)
-	(segment
-		(start 29.25 46.25)
-		(end 31 46)
-		(width 0.25)
-		(layer "F.Cu")
-		(net "+3V3")
-	)
-	(segment
-		(start 35.2 35.52)
-		(end 37 35.52)
-		(width 0.2)
-		(layer "F.Cu")
-		(net "+3V3")
 	)
 	(segment
@@
 	)
 	(segment
-		(start 46.75 40)
-		(end 46.75 38)
-		(width 0.5)
-		(layer "F.Cu")
-		(net "+3V3")
-	)
-	(segment
 		(start 41.93 30.9102)
 		(end 41.93 29.2)
 		(width 0.2)
-		(layer "F.Cu")
-		(net "+3V3")
-	)
-	(segment
-		(start 46.75 38)
-		(end 46 37.75)
-		(width 0.5)
 		(layer "F.Cu")
 		(net "+3V3")
@@
 	)
 	(segment
-		(start 25.5 49)
-		(end 24 45.5)
-		(width 0.5)
-		(layer "F.Cu")
-		(net "+3V3")
-	)
-	(segment
-		(start 37.25 49.75)
-		(end 28.5 50.5)
-		(width 0.25)
-		(layer "F.Cu")
-		(net "+3V3")
-	)
-	(segment
-		(start 24 34.5)
-		(end 29 29.5)
-		(width 0.5)
-		(layer "F.Cu")
-		(net "+3V3")
-	)
-	(segment
 		(start 48.62 38.45)
 		(end 53.45 38.45)
@@
 	)
 	(segment
-		(start 28.5 50.5)
-		(end 27.25 50.5)
-		(width 0.25)
-		(layer "F.Cu")
-		(net "+3V3")
-	)
-	(segment
 		(start 53.45 39.6)
 		(end 53.45 38.45)
@@
 	)
 	(segment
-		(start 37.5 50)
-		(end 27.5 51)
-		(width 0.5)
-		(layer "F.Cu")
-		(net "+3V3")
-	)
-	(segment
-		(start 26 49.25)
-		(end 26.25 48.75)
-		(width 0.25)
-		(layer "F.Cu")
-		(net "+3V3")
-	)
-	(segment
-		(start 33 34.9)
-		(end 33 32.45)
-		(width 0.15)
-		(layer "F.Cu")
-		(net "+3V3")
-	)
-	(segment
 		(start 53.3 39.6)
 		(end 53.25 39.6)
 		(width 0.2)
-		(layer "F.Cu")
-		(net "+3V3")
-	)
-	(segment
-		(start 26.25 48.75)
-		(end 29.25 46.25)
-		(width 0.25)
-		(layer "F.Cu")
-		(net "+3V3")
-	)
-	(segment
-		(start 33 32.45)
-		(end 32.7 32.2)
-		(width 0.15)
-		(layer "F.Cu")
-		(net "+3V3")
-	)
-	(segment
-		(start 32.3 32.05)
-		(end 32.3 31)
-		(width 0.15)
-		(layer "F.Cu")
-		(net "+3V3")
-	)
-	(segment
-		(start 39 48)
-		(end 39 49.5)
-		(width 0.5)
-		(layer "F.Cu")
-		(net "+3V3")
-	)
-	(segment
-		(start 46 40.25)
-		(end 46.75 40)
-		(width 0.5)
-		(layer "F.Cu")
-		(net "+3V3")
-	)
-	(segment
-		(start 24 45.5)
-		(end 24 34.5)
-		(width 0.5)
-		(layer "F.Cu")
-		(net "+3V3")
-	)
-	(segment
-		(start 27.25 50.5)
-		(end 26 49.25)
-		(width 0.25)
-		(layer "F.Cu")
-		(net "+3V3")
-	)
-	(segment
-		(start 39 48)
-		(end 38.75 49.5)
-		(width 0.25)
-		(layer "F.Cu")
-		(net "+3V3")
-	)
-	(segment
-		(start 38.75 49.5)
-		(end 37.25 49.75)
-		(width 0.25)
-		(layer "F.Cu")
-		(net "+3V3")
-	)
-	(segment
-		(start 31 46)
-		(end 32 44.75)
-		(width 0.25)
-		(layer "F.Cu")
-		(net "+3V3")
-	)
-	(segment
-		(start 32.3 35.3)
-		(end 33 34.9)
-		(width 0.15)
-		(layer "F.Cu")
-		(net "+3V3")
-	)
-	(segment
-		(start 27.5 51)
-		(end 25.5 49)
-		(width 0.5)
 		(layer "F.Cu")
 		(net "+3V3")
@@
 	)
 	(segment
-		(start 39 49.5)
-		(end 37.5 50)
-		(width 0.5)
-		(layer "F.Cu")
-		(net "+3V3")
-	)
-	(segment
 		(start 46.9 39.95)
 		(end 45.6 40.25)
@@
 		(net "/power/PWR_LED_K")
 	)
-	(via
-		(at 27.65 38.9)
-		(size 0.6)
-		(drill 0.3)
-		(layers "F.Cu" "B.Cu")
-		(net "VBUS")
-	)
-	(via
-		(at 27.65 44.3)
-		(size 0.6)
-		(drill 0.3)
-		(layers "F.Cu" "B.Cu")
-		(net "VBUS")
-	)
-	(via
-		(at 28.5 38.9)
-		(size 0.6)
-		(drill 0.3)
-		(layers "F.Cu" "B.Cu")
-		(net "VBUS")
-	)
-	(via
-		(at 28.5 44.3)
-		(size 0.6)
-		(drill 0.3)
-		(layers "F.Cu" "B.Cu")
-		(net "VBUS")
-	)
-	(segment
-		(start 28.5 38.9)
-		(end 28.5 44.3)
-		(width 0.8)
-		(layer "B.Cu")
-		(net "VBUS")
-	)
-	(segment
-		(start 27.65 44.3)
-		(end 28.5 44.3)
-		(width 0.8)
-		(layer "B.Cu")
-		(net "VBUS")
-	)
-	(segment
-		(start 27.65 38.9)
-		(end 28.5 38.9)
-		(width 0.8)
-		(layer "B.Cu")
-		(net "VBUS")
-	)
-	(segment
+	(segment
